File: hardware/quadcopter.kicad_pcb (KiCad board)
At the start: 2 copper layers, 33 parts, among them J1 CONN-MOTOR, J2 CONN-MOTOR, J3 CONN-MOTOR, J4 CONN-MOTOR, J5 Conn_ARM_JTAG_SWD_20, J6 GIMBAL, K1 BATTERY, U1 ESC, U2 ESP-WROOM-32-board, U3 LM2936-5.0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

Commit message: [hardware] PCB 1.0
Parts:
- removed J5: Conn_ARM_JTAG_SWD_20, Connector_IDC:IDC-Header_2x10_P2.54mm_Horizontal
- removed JP1: Jumper, Connector_PinHeader_2.54mm:PinHeader_1x02_P2.54mm_Vertical
- C1: footprint Capacitor_THT:CP_Radial_D10.0mm_P5.00mm -> Capacitor_THT:CP_Radial_D5.0mm_P2.50mm
- J1, J2, J3, J4: footprint Connector_PinHeader_2.54mm:PinHeader_1x03_P2.54mm_Vertical -> quadcopter:motor-connector
- K1: footprint Connector_PinHeader_2.54mm:PinHeader_1x02_P2.54mm_Vertical -> quadcopter:battery-connector
- moved R6 124.3 mm to (61.3, 39.0)
- moved K1 123.5 mm to (72.3, 34.3), turned to 270 degrees
- moved R5 117.8 mm to (61.2, 42.5), turned to 180 degrees
- moved U3 115.0 mm to (48.2, 42.7), turned to 180 degrees
- moved R1 112.0 mm to (37.1, 46.0), turned to 90 degrees
- moved C2 108.9 mm to (61.3, 46.0), turned to 180 degrees
- moved C3 108.7 mm to (61.3, 33.7), turned to 90 degrees
- moved D1 108.4 mm to (33.7, 45.9), turned to 90 degrees
- moved C1 101.5 mm to (60.5, 51.8), turned to 180 degrees
- moved J6 101.2 mm to (72.7, 55.4), turned to 180 degrees
- moved R9 100.6 mm to (49.6, 64.2), turned to 90 degrees
- moved R8 96.6 mm to (46.3, 70.1), turned to 90 degrees
- moved R12 93.9 mm to (46.2, 64.2), turned to 270 degrees
- moved U6 93.7 mm to (72.5, 49.4)
- moved R11 88.4 mm to (49.5, 70.1), turned to 270 degrees
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Connections:
- U2 pad 12: TMS -> Net-(U2-Pad12)
- U2 pad 13: TDI -> Net-(U2-Pad13)
- U2 pad 15: TCK -> Net-(U2-Pad15)
- U2 pad 2: ~TRST -> Net-(U2-Pad2)
- U2 pad 23: TDO -> Net-(U2-Pad23)
Routing:
- net GND: track 0.00 -> 391.9 mm, vias 0 -> 122
- net +BATT: track 0.00 -> 139.7 mm, vias 0 -> 12
- net +5V: track 0.00 -> 115.4 mm, vias 0 -> 3
- net ESC_CMD2: track 0.00 -> 109.1 mm
- net ESC_CMD1: track 0.00 -> 108.0 mm, vias 0 -> 2
- net ESC_CMD3: track 0.00 -> 100.5 mm, vias 0 -> 2
- net SCL: track 0.00 -> 94.6 mm, vias 0 -> 1
- net SDA: track 0.00 -> 89.2 mm, vias 0 -> 1
- net GIMBAL_RX: track 0.00 -> 85.3 mm
- net GPS_TX: track 0.00 -> 84.2 mm, vias 0 -> 2
- net HC-SR04_TRIG: track 0.00 -> 73.2 mm
- net Net-(R11-Pad1): track 0.00 -> 68.5 mm, vias 0 -> 4
- net GPS_RX: track 0.00 -> 66.8 mm, vias 0 -> 1
- net +3V3: track 0.00 -> 66.5 mm, vias 0 -> 4
- net SCK: track 0.00 -> 61.9 mm, vias 0 -> 2
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- added copper zone on B.Cu, net GND
- added copper zone on F.Cu, net GND
Other:
- board outline added: 98 x 98 mm
- net class 3.3V added: clearance 0.2, trace_width 0.5, via_dia 0.8, via_drill 0.5
- net class 5V added: clearance 0.5, trace_width 1, via_dia 1.4, via_drill 1
- net class Default: clearance 0.2 -> 0.1; trace_width 0.25 -> 0.5; via_drill 0.4 -> 0.5
- net class GND added: clearance 0.5, trace_width 1, via_dia 1.4, via_drill 1
- net class POWER added: clearance 0.5, trace_width 3, via_dia 1.2, via_drill 0.8
- rule trace_clearance: 0.2 -> 0.1
- rule via_min_size: 0.4 -> 0.6
- board text added: "Quadcopter v1.0"
